Commit message: Update rover_v0.1.urdf

File: rover_v0.1.urdf (robot description, URDF)
Before this commit: robot custom_rover, 9 links, 8 joints
Links:
- added link front_radar; visual box size=0.04 0.18 0.12
- added link top_acrylic; visual box size=1.05 0.65 0.01
Joints:
- added joint chassis_to_front_radar: type fixed, parent chassis, child front_radar, origin xyz=0.52 0 -0.05 rpy=0 0 0

Commit message: Update rover_v0.1.urdf

File: rover_v0.1.urdf (robot description, URDF)
Before this commit: robot custom_rover, 11 links, 9 joints
Links:
- added link front_lidar_body; visual box size=0.1 0.1 0.1
- added link front_lidar_lens; visual cylinder length=0.1 radius=0.05
- added link rear_lidar_body; visual box size=0.1 0.1 0.1
- added link rear_lidar_lens; visual cylinder length=0.1 radius=0.05
Joints:
- removed joint chassis_to_front_radar
- added joint chassis_to_front_lidar: type fixed, parent chassis, child front_lidar_body, origin xyz=0.5 0 0 rpy=0 0 0
- added joint chassis_to_rear_lidar: type fixed, parent chassis, child rear_lidar_body, origin xyz=-0.5 0 0 rpy=0 0 3.14159
- added joint front_lidar_to_lens: type fixed, parent front_lidar_body, child front_lidar_lens, origin xyz=0.02 0 0 rpy=0 1.5708 0
- added joint rear_lidar_to_lens: type fixed, parent rear_lidar_body, child rear_lidar_lens, origin xyz=0.02 0 0 rpy=0 1.5708 0
