Commit message: Update rover_1.urdf

File: rover_1.urdf (robot description, URDF)
Before this commit: robot custom_rover, 9 links, 8 joints
Joints:
- joint fl_wheel_joint: origin xyz=0.35 0.35 -0.05 rpy=-1.5708 0 0 -> xyz=0.35 0.25 -0.05 rpy=-1.5708 0 0
- joint fr_wheel_joint: origin xyz=0.35 -0.35 -0.05 rpy=-1.5708 0 0 -> xyz=0.35 -0.25 -0.05 rpy=-1.5708 0 0
- joint rl_wheel_joint: origin xyz=-0.35 0.35 -0.05 rpy=-1.5708 0 0 -> xyz=-0.35 0.25 -0.05 rpy=-1.5708 0 0
- joint rr_wheel_joint: origin xyz=-0.35 -0.35 -0.05 rpy=-1.5708 0 0 -> xyz=-0.35 -0.25 -0.05 rpy=-1.5708 0 0

Commit message: Update rover_1.urdf

File: rover_1.urdf (robot description, URDF)
Before this commit: robot custom_rover, 9 links, 8 joints
Links:
- removed link front_camera
- added link front_radar; visual box size=0.05 0.15 0.1
Joints:
- removed joint chassis_to_front_camera
- added joint chassis_to_front_radar: type fixed, parent chassis, child front_radar, origin xyz=0.52 0 0.05 rpy=0 0 0

Commit message: Update rover_1.urdf

File: rover_1.urdf (robot description, URDF)
Before this commit: robot custom_rover, 9 links, 8 joints
Links:
- removed link fl_wheel
- removed link fr_wheel
- removed link rl_wheel
- removed link rr_wheel
Joints:
- joint fl_wheel_joint: origin xyz=0.35 0.25 -0.05 rpy=-1.5708 0 0 -> xyz=0.35 0.15 -0.05 rpy=-1.5708 0 0
- joint fr_wheel_joint: origin xyz=0.35 -0.25 -0.05 rpy=-1.5708 0 0 -> xyz=0.35 -0.15 -0.05 rpy=-1.5708 0 0
- joint rl_wheel_joint: origin xyz=-0.35 0.25 -0.05 rpy=-1.5708 0 0 -> xyz=-0.35 0.15 -0.05 rpy=-1.5708 0 0
- joint rr_wheel_joint: origin xyz=-0.35 -0.25 -0.05 rpy=-1.5708 0 0 -> xyz=-0.35 -0.15 -0.05 rpy=-1.5708 0 0
