Commit message: Update rover1.urdf

File: rover1.urdf (robot description, URDF)
Before this commit: robot custom_rover, 9 links, 8 joints
Joints:
- joint fl_wheel_joint: origin xyz=0.35 0.25 -0.05 rpy=-1.5708 0 0 -> xyz=0.35 0.35 -0.05 rpy=-1.5708 0 0
- joint fr_wheel_joint: origin xyz=0.35 -0.25 -0.05 rpy=-1.5708 0 0 -> xyz=0.35 -0.35 -0.05 rpy=-1.5708 0 0
- joint rl_wheel_joint: origin xyz=-0.35 0.25 -0.05 rpy=-1.5708 0 0 -> xyz=-0.35 0.35 -0.05 rpy=-1.5708 0 0
- joint rr_wheel_joint: origin xyz=-0.35 -0.25 -0.05 rpy=-1.5708 0 0 -> xyz=-0.35 -0.35 -0.05 rpy=-1.5708 0 0

Commit message: Update rover1.urdf

File: rover1.urdf (robot description, URDF)
Before this commit: robot custom_rover, 9 links, 8 joints
Joints:
- joint fl_wheel_joint: origin xyz=0.35 0.35 -0.05 rpy=-1.5708 0 0 -> xyz=0.35 0.30 -0.05 rpy=-1.5708 0 0
- joint fr_wheel_joint: origin xyz=0.35 -0.35 -0.05 rpy=-1.5708 0 0 -> xyz=0.35 -0.30 -0.05 rpy=-1.5708 0 0
- joint rl_wheel_joint: origin xyz=-0.35 0.35 -0.05 rpy=-1.5708 0 0 -> xyz=-0.35 0.30 -0.05 rpy=-1.5708 0 0
- joint rr_wheel_joint: origin xyz=-0.35 -0.35 -0.05 rpy=-1.5708 0 0 -> xyz=-0.35 -0.30 -0.05 rpy=-1.5708 0 0

Commit message: Update rover1.urdf

File: rover1.urdf (robot description, URDF)
Before this commit: robot custom_rover, 9 links, 8 joints
Joints:
- joint fl_wheel_joint: origin xyz=0.35 0.30 -0.05 rpy=-1.5708 0 0 -> xyz=0.35 0.28 -0.05 rpy=-1.5708 0 0
- joint fr_wheel_joint: origin xyz=0.35 -0.30 -0.05 rpy=-1.5708 0 0 -> xyz=0.35 -0.28 -0.05 rpy=-1.5708 0 0
- joint rl_wheel_joint: origin xyz=-0.35 0.30 -0.05 rpy=-1.5708 0 0 -> xyz=-0.35 0.28 -0.05 rpy=-1.5708 0 0
- joint rr_wheel_joint: origin xyz=-0.35 -0.30 -0.05 rpy=-1.5708 0 0 -> xyz=-0.35 -0.28 -0.05 rpy=-1.5708 0 0
