Commit message: Update rover3.urdf

File: rover3.urdf (robot description, URDF)
Before this commit: robot custom_rover, 9 links, 8 joints
Joints:
- joint chassis_to_left_lidar: origin xyz=0.1 0.24 0.11 rpy=0 0 0 -> xyz=0.1 0.25 0.11 rpy=0 0 0
- joint chassis_to_right_lidar: origin xyz=0.1 -0.24 0.11 rpy=0 0 0 -> xyz=0.1 -0.25 0.11 rpy=0 0 0

Commit message: Update rover3.urdf

File: rover3.urdf (robot description, URDF)
Before this commit: robot custom_rover, 9 links, 8 joints
Joints:
- joint chassis_to_left_lidar: origin xyz=0.1 0.25 0.11 rpy=0 0 0 -> xyz=0.1 0.255 0.11 rpy=0 0 0
- joint chassis_to_right_lidar: origin xyz=0.1 -0.25 0.11 rpy=0 0 0 -> xyz=0.1 -0.255 0.11 rpy=0 0 0

Commit message: Update rover3.urdf

File: rover3.urdf (robot description, URDF)
Before this commit: robot custom_rover, 9 links, 8 joints
Links:
- added link front_top_lidar; visual box size=0.002 0.118 0.058; visual box size=0.1 0.12 0.06
- added link rear_top_lidar; visual box size=0.002 0.118 0.058; visual box size=0.1 0.12 0.06
Joints:
- added joint chassis_to_front_top_lidar: type fixed, parent chassis, child front_top_lidar, origin xyz=0.4 0 0.13 rpy=0 0 0
- added joint chassis_to_rear_top_lidar: type fixed, parent chassis, child rear_top_lidar, origin xyz=-0.4 0 0.13 rpy=0 0 3.14159

Commit message: Update rover3.urdf

File: rover3.urdf (robot description, URDF)
Before this commit: robot custom_rover, 11 links, 10 joints
Joints:
- joint chassis_to_rear_top_lidar: origin xyz=-0.4 0 0.13 rpy=0 0 3.14159 -> xyz=-0.2 0 0.13 rpy=0 0 3.14159

Commit message: Update rover3.urdf

File: rover3.urdf (robot description, URDF)
Before this commit: robot custom_rover, 11 links, 10 joints
Joints:
- joint chassis_to_front_top_lidar: origin xyz=0.4 0 0.13 rpy=0 0 0 -> xyz=0.15 0 0.13 rpy=0 0 0

Commit message: Update rover3.urdf

File: rover3.urdf (robot description, URDF)
Before this commit: robot custom_rover, 11 links, 10 joints
Joints:
- joint chassis_to_front_top_lidar: origin xyz=0.15 0 0.13 rpy=0 0 0 -> xyz=0.45 0 0.13 rpy=0 0 0
- joint chassis_to_rear_top_lidar: origin xyz=-0.2 0 0.13 rpy=0 0 3.14159 -> xyz=-0.45 0 0.13 rpy=0 0 3.14159

Commit message: Update rover3.urdf

File: rover3.urdf (robot description, URDF)
Before this commit: robot custom_rover, 11 links, 10 joints
Joints:
- joint chassis_to_front_top_lidar: origin xyz=0.45 0 0.13 rpy=0 0 0 -> xyz=0.43 0 0.13 rpy=0 0 0
- joint chassis_to_rear_top_lidar: origin xyz=-0.45 0 0.13 rpy=0 0 3.14159 -> xyz=-0.43 0 0.13 rpy=0 0 3.14159
