Commit message: Update rover4.urdf

File: rover4.urdf (robot description, URDF)
Before this commit: robot custom_rover, 13 links, 12 joints
Links:
- link top_left_lidar: geometry visual box size=0.01 0.06 0.04; visual box size=0.04 0.07 0.06
- link top_right_lidar: geometry visual box size=0.01 0.06 0.04; visual box size=0.04 0.07 0.06
Joints:
- joint chassis_to_top_left_lidar: origin xyz=0.2 0.28 0.13 rpy=0 0 0 -> xyz=0.2 0.28 0.13 rpy=0 0 1.5708
- joint chassis_to_top_right_lidar: origin xyz=0.2 -0.28 0.13 rpy=0 0 0 -> xyz=0.2 -0.28 0.13 rpy=0 0 -1.5708

Commit message: Update rover4.urdf

File: rover4.urdf (robot description, URDF)
Before this commit: robot custom_rover, 13 links, 12 joints
Links:
- link top_left_lidar: geometry visual box size=0.01 0.06 0.02; visual box size=0.04 0.07 0.03
- link top_right_lidar: geometry visual box size=0.01 0.06 0.02; visual box size=0.04 0.07 0.03
Joints:
- joint chassis_to_top_left_lidar: origin xyz=0.2 0.28 0.13 rpy=0 0 1.5708 -> xyz=0.2 0.28 0.115 rpy=0 0 1.5708
- joint chassis_to_top_right_lidar: origin xyz=0.2 -0.28 0.13 rpy=0 0 -1.5708 -> xyz=0.2 -0.28 0.115 rpy=0 0 -1.5708

Commit message: Update rover4.urdf

File: rover4.urdf (robot description, URDF)
Before this commit: robot custom_rover, 13 links, 12 joints
Links:
- removed link front_radar
- removed link front_top_lidar
- removed link left_lidar
- removed link rear_top_lidar
- removed link right_lidar
- removed link top_left_lidar
- removed link top_right_lidar
- added link front_radar_DRVEGRD171 ; visual box size=0.05 0.15 0.1
- added link front_top_lidar_SOSLab_MLX120; visual box size=0.002 0.118 0.058; visual box size=0.1 0.12 0.06
- added link left_lidar_TG30; visual cylinder length=0.03 radius=0.04
- added link rear_top_lidar_SOSLab_MLX120; visual box size=0.002 0.118 0.058; visual box size=0.1 0.12 0.06
- added link right_lidar_TG30; visual cylinder length=0.03 radius=0.04
- added link top_left_lidar_HummingBird_D1; visual box size=0.01 0.06 0.02; visual box size=0.04 0.07 0.03
- added link top_right_lidar_HummingBird_D1; visual box size=0.01 0.06 0.02; visual box size=0.04 0.07 0.03
Joints:
- removed joint chassis_to_front_radar
- removed joint chassis_to_front_top_lidar
- removed joint chassis_to_left_lidar
- removed joint chassis_to_rear_top_lidar
- removed joint chassis_to_right_lidar
- removed joint chassis_to_top_left_lidar
- removed joint chassis_to_top_right_lidar
- added joint chassis_to_front_radar_DRVEGRD171 : type fixed, parent chassis, child front_radar_DRVEGRD171 , origin xyz=0.52 0 0.05 rpy=0 0 0
- added joint chassis_to_front_top_lidar_SOSLab_MLX120: type fixed, parent chassis, child front_top_lidar_SOSLab_MLX120, origin xyz=0.43 0 0.13 rpy=0 0 0
- added joint chassis_to_left_lidar_TG30: type fixed, parent chassis, child left_lidar_TG30, origin xyz=0.1 0.255 0.11 rpy=0 0 0
- added joint chassis_to_rear_top_lidar_SOSLab_MLX120: type fixed, parent chassis, child rear_top_lidar_SOSLab_MLX120, origin xyz=-0.43 0 0.13 rpy=0 0 3.14159
- added joint chassis_to_right_lidar_TG30: type fixed, parent chassis, child right_lidar_TG30, origin xyz=0.1 -0.255 0.11 rpy=0 0 0
- added joint chassis_to_top_left_lidar_HummingBird_D1: type fixed, parent chassis, child top_left_lidar_HummingBird_D1, origin xyz=0.2 0.28 0.115 rpy=0 0 1.5708
- added joint chassis_to_top_right_lidar_HummingBird_D1: type fixed, parent chassis, child top_right_lidar_HummingBird_D1, origin xyz=0.2 -0.28 0.115 rpy=0 0 -1.5708

Commit message: Update rover4.urdf

File: rover4.urdf (robot description, URDF)
Before this commit: robot custom_rover, 13 links, 12 joints
Joints:
- joint chassis_to_left_lidar_TG30: origin xyz=0.1 0.255 0.11 rpy=0 0 0 -> xyz=0.25 0.255 0.11 rpy=0 0 0
- joint chassis_to_right_lidar_TG30: origin xyz=0.1 -0.255 0.11 rpy=0 0 0 -> xyz=0.25 -0.255 0.11 rpy=0 0 0

Commit message: Update rover4.urdf

File: rover4.urdf (robot description, URDF)
Before this commit: robot custom_rover, 13 links, 12 joints
Joints:
- joint chassis_to_left_lidar_TG30: origin xyz=0.25 0.255 0.11 rpy=0 0 0 -> xyz=0.22 0.255 0.11 rpy=0 0 0
- joint chassis_to_right_lidar_TG30: origin xyz=0.25 -0.255 0.11 rpy=0 0 0 -> xyz=0.22 -0.255 0.11 rpy=0 0 0

Commit message: Update rover4.urdf

File: rover4.urdf (robot description, URDF)
Before this commit: robot custom_rover, 13 links, 12 joints
Joints:
- joint chassis_to_left_lidar_TG30: origin xyz=0.22 0.255 0.11 rpy=0 0 0 -> xyz=0.205 0.255 0.11 rpy=0 0 0
- joint chassis_to_right_lidar_TG30: origin xyz=0.22 -0.255 0.11 rpy=0 0 0 -> xyz=0.205 -0.255 0.11 rpy=0 0 0

Commit message: Update rover4.urdf

File: rover4.urdf (robot description, URDF)
Before this commit: robot custom_rover, 13 links, 12 joints
Joints:
- joint chassis_to_left_lidar_TG30: origin xyz=0.205 0.255 0.11 rpy=0 0 0 -> xyz=0.190 0.255 0.11 rpy=0 0 0
- joint chassis_to_right_lidar_TG30: origin xyz=0.205 -0.255 0.11 rpy=0 0 0 -> xyz=0.190 -0.255 0.11 rpy=0 0 0

Commit message: Update rover4.urdf

File: rover4.urdf (robot description, URDF)
Before this commit: robot custom_rover, 13 links, 12 joints
Joints:
- joint chassis_to_left_lidar_TG30: origin xyz=0.190 0.255 0.11 rpy=0 0 0 -> xyz=0.180 0.255 0.11 rpy=0 0 0
- joint chassis_to_right_lidar_TG30: origin xyz=0.190 -0.255 0.11 rpy=0 0 0 -> xyz=0.180 -0.255 0.11 rpy=0 0 0
- joint chassis_to_top_left_lidar_HummingBird_D1: origin xyz=0.2 0.28 0.115 rpy=0 0 1.5708 -> xyz=0.170 0.25 0.115 rpy=0 0 1.5708
- joint chassis_to_top_right_lidar_HummingBird_D1: origin xyz=0.2 -0.28 0.115 rpy=0 0 -1.5708 -> xyz=0.170 -0.25 0.115 rpy=0 0 -1.5708

Commit message: Update rover4.urdf

File: rover4.urdf (robot description, URDF)
Before this commit: robot custom_rover, 13 links, 12 joints
Joints:
- joint chassis_to_top_left_lidar_HummingBird_D1: origin xyz=0.170 0.25 0.115 rpy=0 0 1.5708 -> xyz=0.150 0.23 0.115 rpy=0 0 1.5708
- joint chassis_to_top_right_lidar_HummingBird_D1: origin xyz=0.170 -0.25 0.115 rpy=0 0 -1.5708 -> xyz=0.150 -0.23 0.115 rpy=0 0 -1.5708

Commit message: Update rover4.urdf

File: rover4.urdf (robot description, URDF)
Before this commit: robot custom_rover, 13 links, 12 joints
Joints:
- joint chassis_to_top_left_lidar_HummingBird_D1: origin xyz=0.150 0.23 0.115 rpy=0 0 1.5708 -> xyz=0.120 0.290 0.115 rpy=0 0 1.5708
- joint chassis_to_top_right_lidar_HummingBird_D1: origin xyz=0.150 -0.23 0.115 rpy=0 0 -1.5708 -> xyz=0.120 -0.290 0.115 rpy=0 0 -1.5708

Commit message: Update rover4.urdf

File: rover4.urdf (robot description, URDF)
Before this commit: robot custom_rover, 13 links, 12 joints
Joints:
- joint chassis_to_top_left_lidar_HummingBird_D1: origin xyz=0.120 0.290 0.115 rpy=0 0 1.5708 -> xyz=0.100 0.270 0.115 rpy=0 0 1.5708
- joint chassis_to_top_right_lidar_HummingBird_D1: origin xyz=0.120 -0.290 0.115 rpy=0 0 -1.5708 -> xyz=0.100 -0.270 0.115 rpy=0 0 -1.5708

Commit message: Update rover4.urdf

File: rover4.urdf (robot description, URDF)
Before this commit: robot custom_rover, 13 links, 12 joints
Joints:
- joint chassis_to_top_left_lidar_HummingBird_D1: origin xyz=0.100 0.270 0.115 rpy=0 0 1.5708 -> xyz=0.080 0.265 0.115 rpy=0 0 1.5708
- joint chassis_to_top_right_lidar_HummingBird_D1: origin xyz=0.100 -0.270 0.115 rpy=0 0 -1.5708 -> xyz=0.080 -0.265 0.115 rpy=0 0 -1.5708

Commit message: Update rover4.urdf

File: rover4.urdf (robot description, URDF)
Before this commit: robot custom_rover, 13 links, 12 joints
Joints:
- joint chassis_to_top_left_lidar_HummingBird_D1: origin xyz=0.080 0.265 0.115 rpy=0 0 1.5708 -> xyz=0.070 0.260 0.115 rpy=0 0 1.5708
- joint chassis_to_top_right_lidar_HummingBird_D1: origin xyz=0.080 -0.265 0.115 rpy=0 0 -1.5708 -> xyz=0.070 -0.260 0.115 rpy=0 0 -1.5708

Commit message: Update rover4.urdf

File: rover4.urdf (robot description, URDF)
Before this commit: robot custom_rover, 13 links, 12 joints
Joints:
- joint chassis_to_top_left_lidar_HummingBird_D1: origin xyz=0.070 0.260 0.115 rpy=0 0 1.5708 -> xyz=0.030 0.260 0.115 rpy=0 0 1.5708
- joint chassis_to_top_right_lidar_HummingBird_D1: origin xyz=0.070 -0.260 0.115 rpy=0 0 -1.5708 -> xyz=0.030 -0.260 0.115 rpy=0 0 -1.5708

Commit message: Update rover4.urdf

File: rover4.urdf (robot description, URDF)
Before this commit: robot custom_rover, 13 links, 12 joints
Joints:
- joint chassis_to_left_lidar_TG30: origin xyz=0.180 0.255 0.11 rpy=0 0 0 -> xyz=0.100 0.255 0.11 rpy=0 0 0
- joint chassis_to_right_lidar_TG30: origin xyz=0.180 -0.255 0.11 rpy=0 0 0 -> xyz=0.100 -0.255 0.11 rpy=0 0 0
- joint chassis_to_top_left_lidar_HummingBird_D1: origin xyz=0.030 0.260 0.115 rpy=0 0 1.5708 -> xyz=-0.030 0.260 0.115 rpy=0 0 1.5708
- joint chassis_to_top_right_lidar_HummingBird_D1: origin xyz=0.030 -0.260 0.115 rpy=0 0 -1.5708 -> xyz=-0.030 -0.260 0.115 rpy=0 0 -1.5708

Commit message: Update rover4.urdf

File: rover4.urdf (robot description, URDF)
Before this commit: robot custom_rover, 13 links, 12 joints
Joints:
- joint chassis_to_left_lidar_TG30: origin xyz=0.100 0.255 0.11 rpy=0 0 0 -> xyz=0.050 0.255 0.11 rpy=0 0 0
- joint chassis_to_right_lidar_TG30: origin xyz=0.100 -0.255 0.11 rpy=0 0 0 -> xyz=0.050 -0.255 0.11 rpy=0 0 0

Commit message: Update rover4.urdf

File: rover4.urdf (robot description, URDF)
Before this commit: robot custom_rover, 13 links, 12 joints
Links:
- link left_lidar_TG30: geometry visual cylinder length=0.03 radius=0.03
- link right_lidar_TG30: geometry visual cylinder length=0.03 radius=0.03
Joints:
- joint chassis_to_left_lidar_TG30: origin xyz=0.050 0.255 0.11 rpy=0 0 0 -> xyz=0.070 0.255 0.11 rpy=0 0 0
- joint chassis_to_right_lidar_TG30: origin xyz=0.050 -0.255 0.11 rpy=0 0 0 -> xyz=0.070 -0.255 0.11 rpy=0 0 0

Commit message: Update rover4.urdf

File: rover4.urdf (robot description, URDF)
Before this commit: robot custom_rover, 13 links, 12 joints
Joints:
- joint chassis_to_left_lidar_TG30: origin xyz=0.070 0.255 0.11 rpy=0 0 0 -> xyz=0.060 0.250 0.11 rpy=0 0 0
- joint chassis_to_right_lidar_TG30: origin xyz=0.070 -0.255 0.11 rpy=0 0 0 -> xyz=0.060 -0.250 0.11 rpy=0 0 0

Commit message: Update rover4.urdf

File: rover4.urdf (robot description, URDF)
Before this commit: robot custom_rover, 13 links, 12 joints
Joints:
- joint chassis_to_left_lidar_TG30: origin xyz=0.060 0.250 0.11 rpy=0 0 0 -> xyz=0.060 0.270 0.11 rpy=0 0 0
- joint chassis_to_right_lidar_TG30: origin xyz=0.060 -0.250 0.11 rpy=0 0 0 -> xyz=0.060 -0.270 0.11 rpy=0 0 0

Commit message: Update rover4.urdf

File: rover4.urdf (robot description, URDF)
Before this commit: robot custom_rover, 13 links, 12 joints
Joints:
- joint chassis_to_left_lidar_TG30: origin xyz=0.060 0.270 0.11 rpy=0 0 0 -> xyz=0.050 0.265 0.11 rpy=0 0 0
- joint chassis_to_right_lidar_TG30: origin xyz=0.060 -0.270 0.11 rpy=0 0 0 -> xyz=0.050 -0.265 0.11 rpy=0 0 0
