Commit message: Update rover5.urdf

File: rover5.urdf (robot description, URDF)
Before this commit: robot custom_rover, 13 links, 12 joints
Links:
- removed link top_left_lidar_HummingBird_D1
- removed link top_right_lidar_HummingBird_D1
- added link front_gs2_lidar; visual box size=0.005 0.02 0.015; visual box size=0.005 0.05 0.05
- added link left_gs2_lidar; visual box size=0.005 0.02 0.015; visual box size=0.005 0.05 0.05
- added link rear_gs2_lidar; visual box size=0.005 0.02 0.015; visual box size=0.005 0.05 0.05
- added link right_gs2_lidar; visual box size=0.005 0.02 0.015; visual box size=0.005 0.05 0.05
- link front_top_lidar_SOSLab_MLX120: geometry visual box size=0.1 0.12 0.06
- link rear_top_lidar_SOSLab_MLX120: geometry visual box size=0.1 0.12 0.06
Joints:
- removed joint chassis_to_top_left_lidar_HummingBird_D1
- removed joint chassis_to_top_right_lidar_HummingBird_D1
- added joint chassis_to_front_gs2_lidar: type fixed, parent chassis, child front_gs2_lidar, origin xyz=0.5 0 0 rpy=0 0 0
- added joint chassis_to_left_gs2_lidar: type fixed, parent chassis, child left_gs2_lidar, origin xyz=0 0.3 0 rpy=0 0 1.5708
- added joint chassis_to_rear_gs2_lidar: type fixed, parent chassis, child rear_gs2_lidar, origin xyz=-0.5 0 0 rpy=0 0 3.14159
- added joint chassis_to_right_gs2_lidar: type fixed, parent chassis, child right_gs2_lidar, origin xyz=0 -0.3 0 rpy=0 0 -1.5708
