Commit message: Update rover6.urdf

File: rover6.urdf (robot description, URDF)
Before this commit: robot custom_rover, 13 links, 12 joints
Links:
- added link front_gs2_lidar; visual box size=0.005 0.02 0.015; visual box size=0.005 0.05 0.05
- added link left_gs2_lidar; visual box size=0.005 0.02 0.015; visual box size=0.005 0.05 0.05
- added link rear_gs2_lidar; visual box size=0.005 0.02 0.015; visual box size=0.005 0.05 0.05
- added link right_gs2_lidar; visual box size=0.005 0.02 0.015; visual box size=0.005 0.05 0.05
Joints:
- added joint chassis_to_front_gs2_lidar: type fixed, parent chassis, child front_gs2_lidar, origin xyz=0.5 0 0 rpy=0 0 0
- added joint chassis_to_left_gs2_lidar: type fixed, parent chassis, child left_gs2_lidar, origin xyz=0 0.3 0 rpy=0 0 1.5708
- added joint chassis_to_rear_gs2_lidar: type fixed, parent chassis, child rear_gs2_lidar, origin xyz=-0.5 0 0 rpy=0 0 3.14159
- added joint chassis_to_right_gs2_lidar: type fixed, parent chassis, child right_gs2_lidar, origin xyz=0 -0.3 0 rpy=0 0 -1.5708

Commit message: Update rover6.urdf

File: rover6.urdf (robot description, URDF)
Before this commit: robot custom_rover, 17 links, 16 joints
Links:
- removed link front_gs2_lidar
- removed link rear_gs2_lidar
- removed link right_gs2_lidar
- added link right_gs2_lidar_front; visual box size=0.005 0.02 0.015; visual box size=0.005 0.05 0.05
- added link right_gs2_lidar_rear; visual box size=0.005 0.02 0.015; visual box size=0.005 0.05 0.05
Joints:
- removed joint chassis_to_front_gs2_lidar
- removed joint chassis_to_rear_gs2_lidar
- removed joint chassis_to_right_gs2_lidar
- added joint chassis_to_right_gs2_lidar_front: type fixed, parent chassis, child right_gs2_lidar_front, origin xyz=1.5 -0.1 0 rpy=0 0 -1.5708
- added joint chassis_to_right_gs2_lidar_rear: type fixed, parent chassis, child right_gs2_lidar_rear, origin xyz=-1.5 -0.1 0 rpy=0 0 -1.5708

Commit message: Update rover6.urdf

File: rover6.urdf (robot description, URDF)
Before this commit: robot custom_rover, 16 links, 15 joints
Joints:
- joint chassis_to_right_gs2_lidar_front: origin xyz=1.5 -0.1 0 rpy=0 0 -1.5708 -> xyz=0.3 -0.3 0 rpy=0 0 -1.5708
- joint chassis_to_right_gs2_lidar_rear: origin xyz=-1.5 -0.1 0 rpy=0 0 -1.5708 -> xyz=-0.3 -0.3 0 rpy=0 0 -1.5708

Commit message: Update rover6.urdf

File: rover6.urdf (robot description, URDF)
Before this commit: robot custom_rover, 16 links, 15 joints
Joints:
- joint chassis_to_right_gs2_lidar_front: origin xyz=0.3 -0.3 0 rpy=0 0 -1.5708 -> xyz=0.31 -0.3 0.1 rpy=0 0 -1.5708
- joint chassis_to_right_gs2_lidar_rear: origin xyz=-0.3 -0.3 0 rpy=0 0 -1.5708 -> xyz=-0.31 -0.3 0.1 rpy=0 0 -1.5708

Commit message: Update rover6.urdf

File: rover6.urdf (robot description, URDF)
Before this commit: robot custom_rover, 16 links, 15 joints
Joints:
- joint chassis_to_right_gs2_lidar_front: origin xyz=0.31 -0.3 0.1 rpy=0 0 -1.5708 -> xyz=0.35 -0.3 0.08 rpy=0 0 -1.5708
- joint chassis_to_right_gs2_lidar_rear: origin xyz=-0.31 -0.3 0.1 rpy=0 0 -1.5708 -> xyz=-0.35 -0.3 0.08 rpy=0 0 -1.5708

Commit message: Update rover6.urdf

File: rover6.urdf (robot description, URDF)
Before this commit: robot custom_rover, 16 links, 15 joints
Joints:
- joint chassis_to_right_gs2_lidar_front: origin xyz=0.35 -0.3 0.08 rpy=0 0 -1.5708 -> xyz=0.40 -0.3 0.07 rpy=0 0 -1.5708
- joint chassis_to_right_gs2_lidar_rear: origin xyz=-0.35 -0.3 0.08 rpy=0 0 -1.5708 -> xyz=-0.40 -0.3 0.07 rpy=0 0 -1.5708

Commit message: Update rover6.urdf

File: rover6.urdf (robot description, URDF)
Before this commit: robot custom_rover, 16 links, 15 joints
Joints:
- joint chassis_to_right_gs2_lidar_front: origin xyz=0.40 -0.3 0.07 rpy=0 0 -1.5708 -> xyz=0.43 -0.3 0.07 rpy=0 0 -1.5708
- joint chassis_to_right_gs2_lidar_rear: origin xyz=-0.40 -0.3 0.07 rpy=0 0 -1.5708 -> xyz=-0.43 -0.3 0.07 rpy=0 0 -1.5708

Commit message: Update rover6.urdf

File: rover6.urdf (robot description, URDF)
Before this commit: robot custom_rover, 16 links, 15 joints
Joints:
- joint chassis_to_right_gs2_lidar_front: origin xyz=0.43 -0.3 0.07 rpy=0 0 -1.5708 -> xyz=0.47 -0.3 0.07 rpy=0 0 -1.5708
- joint chassis_to_right_gs2_lidar_rear: origin xyz=-0.43 -0.3 0.07 rpy=0 0 -1.5708 -> xyz=-0.47 -0.3 0.07 rpy=0 0 -1.5708

Commit message: Update rover6.urdf

File: rover6.urdf (robot description, URDF)
Before this commit: robot custom_rover, 16 links, 15 joints
Links:
- removed link left_gs2_lidar
- added link left_gs2_lidar_front; visual box size=0.005 0.02 0.015; visual box size=0.005 0.05 0.05
- added link left_gs2_lidar_rear; visual box size=0.005 0.02 0.015; visual box size=0.005 0.05 0.05
Joints:
- removed joint chassis_to_left_gs2_lidar
- added joint chassis_to_left_gs2_lidar_front: type fixed, parent chassis, child left_gs2_lidar_front, origin xyz=0.47 0.3 0.07 rpy=0 0 1.5708
- added joint chassis_to_left_gs2_lidar_rear: type fixed, parent chassis, child left_gs2_lidar_rear, origin xyz=-0.47 0.3 0.07 rpy=0 0 1.5708
