Commit message: Update rover7.urdf

File: rover7.urdf (robot description, URDF)
Before this commit: robot custom_rover, 17 links, 16 joints
Links:
- added link top_center_cable_trunk; visual cylinder length=0.85 radius=0.012
- added link top_center_gateway; visual box size=0.08 0.09 0.03
- added link top_front_camera; visual box size=0.03 0.04 0.04; visual box size=0.08 0.02 0.002
- added link top_front_left_box; visual box size=0.18 0.08 0.05
- added link top_front_right_box; visual box size=0.18 0.08 0.05
- added link top_left_sensor1; visual box size=0.04 0.025 0.01
- added link top_rear_left_gateway; visual box size=0.03 0.015 0.01; visual box size=0.09 0.05 0.03
- added link top_rear_right_power; visual box size=0.06 0.12 0.03
- added link top_rear_right_switch; visual box size=0.10 0.18 0.04
- added link top_right_sensor1; visual box size=0.04 0.025 0.01
- link right_lidar_TG30: geometry visual cylinder length=0.002 radius=0.015; visual cylinder length=0.03 radius=0.03
Joints:
- added joint chassis_to_cable_trunk: type fixed, parent chassis, child top_center_cable_trunk, origin xyz=0 -0.01 0.106 rpy=0 1.5708 0
- added joint chassis_to_tc_gateway: type fixed, parent chassis, child top_center_gateway, origin xyz=-0.05 0.03 0.115 rpy=0 0 0
- added joint chassis_to_tf_cam: type fixed, parent chassis, child top_front_camera, origin xyz=0.51 0 0.12 rpy=0 0 0
- added joint chassis_to_tfl_box: type fixed, parent chassis, child top_front_left_box, origin xyz=0.38 0.15 0.125 rpy=0 0 0
- added joint chassis_to_tfr_box: type fixed, parent chassis, child top_front_right_box, origin xyz=0.38 -0.15 0.125 rpy=0 0 0
- added joint chassis_to_tl_sensor1: type fixed, parent chassis, child top_left_sensor1, origin xyz=-0.15 0.27 0.105 rpy=0 0 0
- added joint chassis_to_tr_sensor1: type fixed, parent chassis, child top_right_sensor1, origin xyz=-0.15 -0.27 0.105 rpy=0 0 0
- added joint chassis_to_trl_gateway: type fixed, parent chassis, child top_rear_left_gateway, origin xyz=-0.35 0.15 0.115 rpy=0 0 0
- added joint chassis_to_trr_power: type fixed, parent chassis, child top_rear_right_power, origin xyz=-0.40 -0.15 0.115 rpy=0 0 0
- added joint chassis_to_trr_switch: type fixed, parent chassis, child top_rear_right_switch, origin xyz=-0.25 -0.15 0.12 rpy=0 0 0
- joint chassis_to_left_lidar_TG30: origin xyz=0.050 0.265 0.11 rpy=0 0 0 -> xyz=0.050 0.285 0.11 rpy=0 0 0
- joint chassis_to_right_lidar_TG30: origin xyz=0.050 -0.265 0.11 rpy=0 0 0 -> xyz=0.050 -0.285 0.11 rpy=0 0 0

Commit message: Update rover7.urdf

File: rover7.urdf (robot description, URDF)
Before this commit: robot custom_rover, 27 links, 26 joints
Links:
- removed link top_front_left_box
Joints:
- removed joint chassis_to_tfl_box

Commit message: Update rover7.urdf

File: rover7.urdf (robot description, URDF)
Before this commit: robot custom_rover, 26 links, 25 joints
Links:
- added link top_front_left_box; visual box size=0.08 0.18 0.05
- link top_front_right_box: geometry visual box size=0.08 0.18 0.05
Joints:
- added joint chassis_to_tfl_box: type fixed, parent chassis, child top_front_left_box, origin xyz=0.38 0.15 0.125 rpy=0 0 0

Commit message: Update rover7.urdf

File: rover7.urdf (robot description, URDF)
Before this commit: robot custom_rover, 27 links, 26 joints
Links:
- link front_top_lidar_SOSLab_MLX120: geometry visual box size=0.002 0.118 0.058; visual box size=0.08 0.12 0.06

Commit message: Update rover7.urdf

File: rover7.urdf (robot description, URDF)
Before this commit: robot custom_rover, 27 links, 26 joints
Links:
- link front_top_lidar_SOSLab_MLX120: geometry visual box size=0.002 0.118 0.058; visual box size=0.0667 0.12 0.06

Commit message: Update rover7.urdf

File: rover7.urdf (robot description, URDF)
Before this commit: robot custom_rover, 27 links, 26 joints
Links:
- link rear_top_lidar_SOSLab_MLX120: geometry visual box size=0.002 0.118 0.058; visual box size=0.0667 0.12 0.06
Joints:
- joint chassis_to_front_top_lidar_SOSLab_MLX120: origin xyz=0.43 0 0.13 rpy=0 0 0 -> xyz=0.45 0 0.13 rpy=0 0 0
- joint chassis_to_rear_top_lidar_SOSLab_MLX120: origin xyz=-0.43 0 0.13 rpy=0 0 3.14159 -> xyz=-0.45 0 0.13 rpy=0 0 3.14159

Commit message: Update rover7.urdf

File: rover7.urdf (robot description, URDF)
Before this commit: robot custom_rover, 27 links, 26 joints
Links:
- removed link top_center_cable_trunk
Joints:
- removed joint chassis_to_cable_trunk
- joint chassis_to_tfl_box: origin xyz=0.38 0.15 0.125 rpy=0 0 0 -> xyz=0.35 0.15 0.125 rpy=0 0 0
- joint chassis_to_tfr_box: origin xyz=0.38 -0.15 0.125 rpy=0 0 0 -> xyz=0.35 -0.15 0.125 rpy=0 0 0

Commit message: Update rover7.urdf

File: rover7.urdf (robot description, URDF)
Before this commit: robot custom_rover, 26 links, 25 joints
Links:
- link left_lidar_TG30: geometry visual cylinder length=0.002 radius=0.015; visual cylinder length=0.03 radius=0.03
Joints:
- joint chassis_to_front_top_lidar_SOSLab_MLX120: origin xyz=0.45 0 0.13 rpy=0 0 0 -> xyz=0.43 0.2 0.13 rpy=0 0 0
- joint chassis_to_left_lidar_TG30: origin xyz=0.050 0.285 0.11 rpy=0 0 0 -> xyz=0.040 0.285 0.11 rpy=0 0 0
- joint chassis_to_right_lidar_TG30: origin xyz=0.050 -0.285 0.11 rpy=0 0 0 -> xyz=0.040 -0.285 0.11 rpy=0 0 0

Commit message: Update rover7.urdf

File: rover7.urdf (robot description, URDF)
Before this commit: robot custom_rover, 26 links, 25 joints
Joints:
- joint chassis_to_left_lidar_TG30: origin xyz=0.040 0.285 0.11 rpy=0 0 0 -> xyz=0.030 0.285 0.11 rpy=0 0 0
- joint chassis_to_right_lidar_TG30: origin xyz=0.040 -0.285 0.11 rpy=0 0 0 -> xyz=0.030 -0.285 0.11 rpy=0 0 0

Commit message: Update rover7.urdf

File: rover7.urdf (robot description, URDF)
Before this commit: robot custom_rover, 26 links, 25 joints
Joints:
- joint chassis_to_left_lidar_TG30: origin xyz=0.030 0.285 0.11 rpy=0 0 0 -> xyz=0.050 0.270 0.11 rpy=0 0 0
- joint chassis_to_right_lidar_TG30: origin xyz=0.030 -0.285 0.11 rpy=0 0 0 -> xyz=0.050 -0.270 0.11 rpy=0 0 0

Commit message: Update rover7.urdf

File: rover7.urdf (robot description, URDF)
Before this commit: robot custom_rover, 26 links, 25 joints
Joints:
- joint chassis_to_left_lidar_TG30: origin xyz=0.050 0.270 0.11 rpy=0 0 0 -> xyz=0.050 0.265 0.11 rpy=0 0 0
- joint chassis_to_right_lidar_TG30: origin xyz=0.050 -0.270 0.11 rpy=0 0 0 -> xyz=0.050 -0.265 0.11 rpy=0 0 0

Commit message: Update rover7.urdf

File: rover7.urdf (robot description, URDF)
Before this commit: robot custom_rover, 26 links, 25 joints
Links:
- link top_front_left_box: geometry visual box size=0.08 0.22 0.05
- link top_front_right_box: geometry visual box size=0.08 0.22 0.05

Commit message: Update rover7.urdf

File: rover7.urdf (robot description, URDF)
Before this commit: robot custom_rover, 26 links, 25 joints
Links:
- link top_front_left_box: geometry visual box size=0.08 0.25 0.05
- link top_front_right_box: geometry visual box size=0.08 0.25 0.05

Commit message: Update rover7.urdf

File: rover7.urdf (robot description, URDF)
Before this commit: robot custom_rover, 26 links, 25 joints
Links:
- link top_front_left_box: geometry visual box size=0.08 0.24 0.05
- link top_front_right_box: geometry visual box size=0.08 0.24 0.05
Joints:
- joint chassis_to_tfl_box: origin xyz=0.35 0.15 0.125 rpy=0 0 0 -> xyz=0.35 0.13 0.125 rpy=0 0 0
- joint chassis_to_tfr_box: origin xyz=0.35 -0.15 0.125 rpy=0 0 0 -> xyz=0.35 -0.13 0.125 rpy=0 0 0

Commit message: Update rover7.urdf

File: rover7.urdf (robot description, URDF)
Before this commit: robot custom_rover, 26 links, 25 joints
Links:
- link top_front_left_box: geometry visual box size=0.08 0.23 0.05
- link top_front_right_box: geometry visual box size=0.08 0.23 0.05

Commit message: Update rover7.urdf

File: rover7.urdf (robot description, URDF)
Before this commit: robot custom_rover, 26 links, 25 joints
Joints:
- joint chassis_to_tf_cam: origin xyz=0.51 0 0.12 rpy=0 0 0 -> xyz=0.46 -0.2 0.12 rpy=0 0 0

Commit message: Update rover7.urdf

File: rover7.urdf (robot description, URDF)
Before this commit: robot custom_rover, 26 links, 25 joints
Joints:
- joint chassis_to_tf_cam: origin xyz=0.46 -0.2 0.12 rpy=0 0 0 -> xyz=0.48 -0.02 0.12 rpy=0 0 0

Commit message: Update rover7.urdf

File: rover7.urdf (robot description, URDF)
Before this commit: robot custom_rover, 26 links, 25 joints
Joints:
- joint chassis_to_front_top_lidar_SOSLab_MLX120: origin xyz=0.43 0.2 0.13 rpy=0 0 0 -> xyz=0.45 0.05 0.13 rpy=0 0 0
- joint chassis_to_tf_cam: origin xyz=0.48 -0.02 0.12 rpy=0 0 0 -> xyz=0.48 -0.03 0.12 rpy=0 0 0

Commit message: Update rover7.urdf

File: rover7.urdf (robot description, URDF)
Before this commit: robot custom_rover, 26 links, 25 joints
Joints:
- joint chassis_to_front_top_lidar_SOSLab_MLX120: origin xyz=0.45 0.05 0.13 rpy=0 0 0 -> xyz=0.44 0.07 0.13 rpy=0 0 0
- joint chassis_to_tf_cam: origin xyz=0.48 -0.03 0.12 rpy=0 0 0 -> xyz=0.48 -0.04 0.12 rpy=0 0 0

Commit message: Update rover7.urdf

File: rover7.urdf (robot description, URDF)
Before this commit: robot custom_rover, 26 links, 25 joints
Joints:
- joint chassis_to_rear_top_lidar_SOSLab_MLX120: origin xyz=-0.45 0 0.13 rpy=0 0 3.14159 -> xyz=-0.44 0.07 0.13 rpy=0 0 3.14159
- joint chassis_to_tf_cam: origin xyz=0.48 -0.04 0.12 rpy=0 0 0 -> xyz=0.48 -0.05 0.12 rpy=0 0 0

Commit message: Update rover7.urdf

File: rover7.urdf (robot description, URDF)
Before this commit: robot custom_rover, 26 links, 25 joints
Links:
- removed link top_left_sensor1
- removed link top_right_sensor1
- added link top_rear_camera; visual box size=0.03 0.04 0.04; visual box size=0.08 0.02 0.002
Joints:
- removed joint chassis_to_tl_sensor1
- removed joint chassis_to_tr_sensor1
- joint chassis_to_tf_cam: child top_front_camera -> top_rear_camera; origin xyz=0.48 -0.05 0.12 rpy=0 0 0 -> xyz=0.51 0 0.12 rpy=0 0 3.14159

Commit message: Update rover7.urdf

File: rover7.urdf (robot description, URDF)
Before this commit: robot custom_rover, 25 links, 23 joints
Joints:
- removed joint chassis_to_tf_cam
- added joint chassis_to_top_front_camera: type fixed, parent chassis, child top_front_camera, origin xyz=0.48 -0.05 0.12 rpy=0 0 0
- added joint chassis_to_top_rear_camera: type fixed, parent chassis, child top_rear_camera, origin xyz=-0.48 -0.05 0.12 rpy=0 0 3.14159

Commit message: Update rover7.urdf

File: rover7.urdf (robot description, URDF)
Before this commit: robot custom_rover, 25 links, 24 joints
Joints:
- joint chassis_to_front_top_lidar_SOSLab_MLX120: origin xyz=0.44 0.07 0.13 rpy=0 0 0 -> xyz=0.46 0.07 0.13 rpy=0 0 0
- joint chassis_to_rear_top_lidar_SOSLab_MLX120: origin xyz=-0.44 0.07 0.13 rpy=0 0 3.14159 -> xyz=-0.46 0.07 0.13 rpy=0 0 3.14159
