Commit message: Update rover8.urdf

File: rover8.urdf (robot description, URDF)
Before this commit: robot custom_rover, 25 links, 24 joints
Links:
- removed link top_front_left_box
- removed link top_front_right_box
- removed link top_rear_right_power
- added link top_front_left_box_RPiv5; visual box size=0.08 0.23 0.05
- added link top_front_right_boxRPiv5; visual box size=0.08 0.23 0.05
Joints:
- removed joint chassis_to_trr_power
- joint chassis_to_tfl_box: child top_front_left_box -> top_front_left_box_RPiv5
- joint chassis_to_tfr_box: child top_front_right_box -> top_front_right_box_RPiv5

Commit message: Update rover8.urdf

File: rover8.urdf (robot description, URDF)
Before this commit: robot custom_rover, 24 links, 23 joints
Links:
- removed link top_center_gateway
- removed link top_front_right_boxRPiv5
- removed link top_rear_left_gateway
- added link top_front_PoE_gateway; visual box size=0.08 0.09 0.03
- added link top_front_right_box_RPiv5; visual box size=0.08 0.23 0.05
- added link top_rear_CANgateway_RearCAM; visual box size=0.03 0.015 0.01; visual box size=0.09 0.05 0.03
Joints:
- joint chassis_to_tc_gateway: child top_center_gateway -> top_front_PoE_gateway; origin xyz=-0.05 0.03 0.115 rpy=0 0 0 -> xyz=0.2 0.03 0.115 rpy=0 0 0
- joint chassis_to_trl_gateway: child top_rear_left_gateway -> top_rear_CANgateway_RearCAM; origin xyz=-0.35 0.15 0.115 rpy=0 0 0 -> xyz=-0.35 -0.05 0.115 rpy=0 0 0

Commit message: Update rover8.urdf

File: rover8.urdf (robot description, URDF)
Before this commit: robot custom_rover, 24 links, 23 joints
Links:
- link top_rear_CANgateway_RearCAM: geometry visual box size=0.09 0.05 0.03
Joints:
- joint chassis_to_tc_gateway: origin xyz=0.2 0.03 0.115 rpy=0 0 0 -> xyz=0.1 -0.1 0.115 rpy=0 0 0
- joint chassis_to_trl_gateway: origin xyz=-0.35 -0.05 0.115 rpy=0 0 0 -> xyz=-0.37 -0.05 0.115 rpy=0 0 0

Commit message: Update rover8.urdf

File: rover8.urdf (robot description, URDF)
Before this commit: robot custom_rover, 24 links, 23 joints
Links:
- link top_rear_CANgateway_RearCAM: geometry visual box size=0.06 0.04 0.03
Joints:
- joint chassis_to_trl_gateway: origin xyz=-0.37 -0.05 0.115 rpy=0 0 0 -> xyz=-0.39 -0.05 0.115 rpy=0 0 0

Commit message: Update rover8.urdf

File: rover8.urdf (robot description, URDF)
Before this commit: robot custom_rover, 24 links, 23 joints
Links:
- removed link top_rear_right_switch
- added link top_rear_2.5Gbps_switch; visual box size=0.10 0.20 0.04
Joints:
- joint chassis_to_trr_switch: child top_rear_right_switch -> top_rear_2.5Gbps_switch; origin xyz=-0.25 -0.15 0.12 rpy=0 0 0 -> xyz=-0.30 0.20 0.12 rpy=0 0 0

Commit message: Update rover8.urdf

File: rover8.urdf (robot description, URDF)
Before this commit: robot custom_rover, 24 links, 23 joints
Joints:
- joint chassis_to_trr_switch: origin xyz=-0.30 0.20 0.12 rpy=0 0 0 -> xyz=-0.30 0.12 0.12 rpy=0 0 0

Commit message: Update rover8.urdf

File: rover8.urdf (robot description, URDF)
Before this commit: robot custom_rover, 24 links, 23 joints
Links:
- link top_front_PoE_gateway: geometry visual box size=0.08 0.10 0.03
Joints:
- joint chassis_to_tc_gateway: origin xyz=0.1 -0.1 0.115 rpy=0 0 0 -> xyz=0.1 -0.05 0.115 rpy=0 0 0

Commit message: Update rover8.urdf

File: rover8.urdf (robot description, URDF)
Before this commit: robot custom_rover, 24 links, 23 joints
Joints:
- joint chassis_to_tc_gateway: origin xyz=0.1 -0.05 0.115 rpy=0 0 0 -> xyz=0.1 -0.08 0.115 rpy=0 0 0
