Commit message: Update rover9.urdf

File: rover9.urdf (robot description, URDF)
Before this commit: robot custom_rover, 24 links, 23 joints
Links:
- added link insung_transceiver; visual box size=0.12 0.10 0.03; visual cylinder length=0.01 radius=0.003
- added link moonwalker_imu; visual box size=0.04 0.04 0.01
Joints:
- added joint chassis_to_imu: type fixed, parent chassis, child moonwalker_imu, origin xyz=0.0 0.0 0.105 rpy=0 0 0
- added joint chassis_to_insung: type fixed, parent chassis, child insung_transceiver, origin xyz=-0.15 0.0 0.115 rpy=0 0 0

Commit message: Update rover9.urdf

File: rover9.urdf (robot description, URDF)
Before this commit: robot custom_rover, 26 links, 25 joints
Joints:
- joint chassis_to_imu: origin xyz=0.0 0.0 0.105 rpy=0 0 0 -> xyz=0.3 -0.14 0.105 rpy=0 0 0
- joint chassis_to_insung: origin xyz=-0.15 0.0 0.115 rpy=0 0 0 -> xyz=0.2 -0.13 0.115 rpy=0 0 0

Commit message: Update rover9.urdf

File: rover9.urdf (robot description, URDF)
Before this commit: robot custom_rover, 26 links, 25 joints
Links:
- link insung_transceiver: geometry visual box size=0.8 0.6 0.03; visual cylinder length=0.01 radius=0.003
Joints:
- joint chassis_to_imu: origin xyz=0.3 -0.14 0.105 rpy=0 0 0 -> xyz=0.2 0.16 0.105 rpy=0 0 0
- joint chassis_to_insung: origin xyz=0.2 -0.13 0.115 rpy=0 0 0 -> xyz=0.2 0.13 0.115 rpy=0 0 0

Commit message: Update rover9.urdf

File: rover9.urdf (robot description, URDF)
Before this commit: robot custom_rover, 26 links, 25 joints
Links:
- link insung_transceiver: geometry visual box size=0.08 0.06 0.03; visual cylinder length=0.01 radius=0.003

Commit message: Update rover9.urdf

File: rover9.urdf (robot description, URDF)
Before this commit: robot custom_rover, 26 links, 25 joints
Joints:
- joint chassis_to_insung: origin xyz=0.2 0.13 0.115 rpy=0 0 0 -> xyz=0.2 0.03 0.115 rpy=0 0 0

Commit message: Update rover9.urdf

File: rover9.urdf (robot description, URDF)
Before this commit: robot custom_rover, 26 links, 25 joints
Joints:
- joint chassis_to_insung: origin xyz=0.2 0.03 0.115 rpy=0 0 0 -> xyz=0.2 0.035 0.115 rpy=0 0 0

Commit message: Update rover9.urdf

File: rover9.urdf (robot description, URDF)
Before this commit: robot custom_rover, 26 links, 25 joints
Joints:
- joint chassis_to_insung: origin xyz=0.2 0.035 0.115 rpy=0 0 0 -> xyz=0.2 0.040 0.115 rpy=0 0 0

Commit message: Update rover9.urdf

File: rover9.urdf (robot description, URDF)
Before this commit: robot custom_rover, 26 links, 25 joints
Joints:
- joint chassis_to_insung: origin xyz=0.2 0.040 0.115 rpy=0 0 0 -> xyz=0.2 0.050 0.115 rpy=0 0 0

Commit message: Update rover9.urdf

File: rover9.urdf (robot description, URDF)
Before this commit: robot custom_rover, 26 links, 25 joints
Joints:
- joint chassis_to_imu: origin xyz=0.2 0.16 0.105 rpy=0 0 0 -> xyz=0.24 0.16 0.105 rpy=0 0 0

Commit message: Update rover9.urdf

File: rover9.urdf (robot description, URDF)
Before this commit: robot custom_rover, 26 links, 25 joints
Joints:
- joint chassis_to_imu: origin xyz=0.24 0.16 0.105 rpy=0 0 0 -> xyz=0.22 0.16 0.105 rpy=0 0 0
- joint chassis_to_insung: origin xyz=0.2 0.050 0.115 rpy=0 0 0 -> xyz=0.2 0.060 0.115 rpy=0 0 0
