Commit message: Update roverModel_v1.0.urdf

File: roverModel_v1.0.urdf (robot description, URDF)
Before this commit: robot custom_rover, 26 links, 25 joints
Links:
- added link wire_harness; visual box size=0.01 0.05 0.01; visual box size=0.01 0.05 0.01
Joints:
- added joint chassis_to_wire_harness: type fixed, parent chassis, child wire_harness, origin xyz=0 0 0.105 rpy=0 0 0

Commit message: Update roverModel_v1.0.urdf

File: roverModel_v1.0.urdf (robot description, URDF)
Before this commit: robot custom_rover, 27 links, 26 joints
Links:
- removed link wire_harness
Joints:
- removed joint chassis_to_wire_harness

Commit message: Update roverModel_v1.0.urdf

File: roverModel_v1.0.urdf (robot description, URDF)
Before this commit: robot custom_rover, 26 links, 25 joints
Joints:
- removed joint chassis_to_insung

Commit message: Update roverModel_v1.0.urdf

File: roverModel_v1.0.urdf (robot description, URDF)
Before this commit: robot custom_rover, 26 links, 24 joints
Joints:
- added joint chassis_to_insung: type fixed, parent chassis, child insung_transceiver, origin xyz=0.2 0.060 0.115 rpy=0 0 0

Commit message: Update roverModel_v1.0.urdf

File: roverModel_v1.0.urdf (robot description, URDF)
Before this commit: robot custom_rover, 26 links, 25 joints
Links:
- link front_radar_DRVEGRD171 : geometry visual box size=0.05 0.15 0.02; visual box size=0.055 0.155 0.002

Commit message: Update roverModel_v1.0.urdf

File: roverModel_v1.0.urdf (robot description, URDF)
Before this commit: robot custom_rover, 26 links, 25 joints
Joints:
- joint chassis_to_front_radar_DRVEGRD171 : origin xyz=0.52 0 0.05 rpy=0 0 0 -> xyz=0.52 0 0.05 rpy=0 1.5708 0

Commit message: Update roverModel_v1.0.urdf

File: roverModel_v1.0.urdf (robot description, URDF)
Before this commit: robot custom_rover, 26 links, 25 joints
Joints:
- joint chassis_to_front_radar_DRVEGRD171 : origin xyz=0.52 0 0.05 rpy=0 1.5708 0 -> xyz=0.50 0 0.05 rpy=0 1.5708 0

Commit message: Update roverModel_v1.0.urdf

File: roverModel_v1.0.urdf (robot description, URDF)
Before this commit: robot custom_rover, 26 links, 25 joints
Links:
- link front_radar_DRVEGRD171 : geometry visual box size=0.055 0.155 0.002; visual box size=0.06 0.10 0.02

Commit message: Update roverModel_v1.0.urdf

File: roverModel_v1.0.urdf (robot description, URDF)
Before this commit: robot custom_rover, 26 links, 25 joints
Links:
- link front_radar_DRVEGRD171 : geometry visual box size=0.06 0.10 0.02; visual box size=0.065 0.105 0.002

Commit message: Update roverModel_v1.0.urdf

File: roverModel_v1.0.urdf (robot description, URDF)
Before this commit: robot custom_rover, 26 links, 25 joints
Links:
- link front_top_lidar_SOSLab_MLX120: geometry visual box size=0.0012 0.0708 0.0348; visual box size=0.04002 0.072 0.036

Commit message: Update roverModel_v1.0.urdf

File: roverModel_v1.0.urdf (robot description, URDF)
Before this commit: robot custom_rover, 26 links, 25 joints
Links:
- link front_top_lidar_SOSLab_MLX120: geometry visual box size=0.0026 0.1534 0.0754; visual box size=0.08671 0.156 0.078

Commit message: Update roverModel_v1.0.urdf

File: roverModel_v1.0.urdf (robot description, URDF)
Before this commit: robot custom_rover, 26 links, 25 joints
Links:
- removed link rear_top_lidar_SOSLab_MLX120
- link front_top_lidar_SOSLab_MLX120: geometry visual box size=0.0016 0.0944 0.0464; visual box size=0.05336 0.096 0.048
Joints:
- removed joint chassis_to_front_top_lidar_SOSLab_MLX120

Commit message: Update roverModel_v1.0.urdf

File: roverModel_v1.0.urdf (robot description, URDF)
Before this commit: robot custom_rover, 25 links, 24 joints
Links:
- added link rear_top_lidar_SOSLab_MLX120; visual box size=0.002 0.118 0.058; visual box size=0.0667 0.12 0.06
- link front_top_lidar_SOSLab_MLX120: geometry visual box size=0.002 0.118 0.058; visual box size=0.0667 0.12 0.06
Joints:
- added joint chassis_to_front_top_lidar_SOSLab_MLX120: type fixed, parent chassis, child front_top_lidar_SOSLab_MLX120, origin xyz=0.46 0.07 0.13 rpy=0 0 0

Commit message: Update roverModel_v1.0.urdf

File: roverModel_v1.0.urdf (robot description, URDF)
Before this commit: robot custom_rover, 26 links, 25 joints
Links:
- removed link top_left_lidar_HummingBird_D1
- added link d1_101_link; visual box size=0.01 0.06 0.02; visual box size=0.04 0.07 0.03
Joints:
- joint chassis_to_top_left_lidar_HummingBird_D1: child top_left_lidar_HummingBird_D1 -> d1_101_link

Commit message: Update roverModel_v1.0.urdf

File: roverModel_v1.0.urdf (robot description, URDF)
Before this commit: robot custom_rover, 26 links, 25 joints
Links:
- removed link d1_101_link
- added link top_left_lidar_HummingBird_D1; visual box size=0.01 0.06 0.02; visual box size=0.04 0.07 0.03
Joints:
- joint chassis_to_top_left_lidar_HummingBird_D1: child d1_101_link -> top_left_lidar_HummingBird_D1

Commit message: Update roverModel_v1.0.urdf

File: roverModel_v1.0.urdf (robot description, URDF)
Before this commit: robot custom_rover, 26 links, 25 joints
Joints:
- joint chassis_to_top_left_lidar_HummingBird_D1: origin xyz=-0.030 0.260 0.115 rpy=0 0 1.5708 -> xyz=-0.030 0.260 0.05 rpy=0 0 1.5708
- joint chassis_to_top_right_lidar_HummingBird_D1: origin xyz=-0.030 -0.260 0.115 rpy=0 0 -1.5708 -> xyz=-0.030 -0.260 0.05 rpy=0 0 -1.5708

Commit message: Update roverModel_v1.0.urdf

File: roverModel_v1.0.urdf (robot description, URDF)
Before this commit: robot custom_rover, 26 links, 25 joints
Joints:
- joint chassis_to_top_left_lidar_HummingBird_D1: origin xyz=-0.030 0.260 0.05 rpy=0 0 1.5708 -> xyz=-0.030 0.260 0.115 rpy=0 0 1.5708
- joint chassis_to_top_right_lidar_HummingBird_D1: origin xyz=-0.030 -0.260 0.05 rpy=0 0 -1.5708 -> xyz=-0.030 -0.260 0.115 rpy=0 0 -1.5708
